File: Connector.kicad_sch (KiCad schematic)
At the start: 13 parts, among them J1 TC2070-IDC-NL, J10 SM02B-GHS-TB, J11 Conn_01x06, J2 XT30PW-M, J3 SM04B-GHS-TB, J4 SM02B-GHS-TB, J5 BM02B-GHS-TBT, J6 SM02B-GHS-TB, J7 SM02B-GHS-TB, J8 SM03B-GHS-TB, J9 SM04B-GHS-TB, SW2 OS102011MA1Q, U8 TPD4E05U06DQA

Commit message: feat: add SPI connector and I²c pull up for magnetic encoder
Parts:
- added R85, R86: 10K, Resistor_SMD:R_0603_1608Metric, symbol Device:R_Small
Connections:
- net +3V3: now also R85.2, R86.2
- net NSS_MCU: now also R86.1
- net SCK_MCU: now also R85.1
Other:
- note added: "Pull Up I²C/SPI"
- note added: "Pull up for I²C open drain circuit"
- moved on the sheet: J11, J3, J4, J5, J6, J7, J8, J9

Commit message: feat: finalize STM32G070CBT6 LQFP48 pinout and peripheral mapping
Parts:
- added J12: SM02B-GHS-TB, Connector_JST:JST_GH_SM02B-GHS-TB_1x02-1MP_P1.25mm_Horizontal, symbol Connector_Generic:Conn_01x02
- added J13: XT30PW-M, KineticCore:AMASS_XT30PW-M, symbol KineticCore:XT30PW-M
- J5: footprint Connector_JST:JST_XH_S2B-XH-A_1x02_P2.50mm_Horizontal -> Connector_JST:JST_GH_SM02B-GHS-TB_1x02-1MP_P1.25mm_Horizontal
- R85, R86: value 10K -> 4K7
Connections:
- net GND: now also J12.2 (Pin_2)
- new net NFAULT_EXT: J12.1 (Pin_1)
- new net OUT_A_EXT: J13.P
- new net OUT_B_EXT: J13.N
Other:
- note added: "Motor"
- note added: "Optional Open-Drain Termination for Hybrid SPI/I²C Interface"
- note added: "Power Fault"
- note added: "Supply"
- note removed: "Pull up for I²C open drain circuit"
- moved on the sheet: J11, J2, J3, J4, J5, J6, J7, J8, J9, R85, R86
