File: Interface.kicad_sch (KiCad schematic)
At the start: 67 parts, among them U20 74LVC2G126, U22 SN74LVC2G14DBV, U3 THVD1400D, U4 SN74LVC2G14DBV, U6 USBLC6-2SC6, U7 TLP2310, U9 TLP2310

Commit message: feat: finalize STM32G070CBT6 LQFP48 pinout and peripheral mapping
Other:
- note added: "UART N°1 activity LED indicators (pulse stretcher)"
- note added: "UART N°2 activity LED indicators (pulse stretcher)"
- note removed: "UART activity LED indicators (pulse stretcher)"
Changed lines of the file:
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@@
 		)
 	)
-	(text "UART activity LED indicators (pulse stretcher)"
+	(text "UART N°1 activity LED indicators (pulse stretcher)"
 		(exclude_from_sim no)
-		(at 45.974 16.764 0)
+		(at 49.276 16.764 0)
 		(effects
 			(font
@@
 		)
 	)
-	(text "UART activity LED indicators (pulse stretcher)"
+	(text "UART N°2 activity LED indicators (pulse stretcher)"
 		(exclude_from_sim no)
-		(at 45.974 67.31 0)
+		(at 49.276 67.564 0)
 		(effects
 			(font
